Commit message: master thesis

File: cvg_sim_gazebo/urdf/quadrotor_base.urdf.xacro (robot description, xacro)
@@ -11,4 +11,7 @@
     <link name="base_link">
       <inertial>
+        <!-- <mass value="0.380" />
+        <origin xyz="0 0 0" />
+        <inertia ixx="0.0095" ixy="0.0" ixz="0.0" iyy="0.0185" iyz="0.0" izz="0.0255" /> -->
         <mass value="1.477" />
         <origin xyz="0 0 0" />
